File: Headunit/HW_Headunit/Board/HW_Headunit.kicad_sch (KiCad schematic)
At the start: 4 parts, among them J1 AudioJack4_SwitchT1, J2 AudioJack4_SwitchT1, J3 2328702-8, U2 PY32F002AW15U

Commit message: Exported fabrication files
Parts:
- removed U2: PY32F002AW15U, Package_DFN_QFN:QFN-16-1EP_3x3mm_P0.5mm_EP1.7x1.7mm, symbol USER:PY32F002AW15U
- added C1, C4, C6, C73: 1u, Capacitor_SMD:C_0603_1608Metric, symbol Device:C
- added C2, C3, C5, C68, C7: 100n, Capacitor_SMD:C_0402_1005Metric, symbol Device:C
- added D1: SP0502BAHT, Package_TO_SOT_SMD:SOT-23, symbol Power_Protection:SP0502BAHT
- added F1: 0603L020YR, Fuse:Fuse_0603_1608Metric, symbol Device:Polyfuse
- added J4: HS096T01H13, USER:HS096T01H13, symbol Connector_Generic:Conn_01x13
- added J5: Conn_01x05, Connector_PinHeader_2.54mm:PinHeader_1x05_P2.54mm_Vertical, symbol Connector_Generic:Conn_01x05
- added Q2, Q3: DMC2400UV, Package_TO_SOT_SMD:SOT-563, symbol USER:DMC2400UV
- added R1, R2: 62R, Resistor_SMD:R_0805_2012Metric, symbol Device:R
- added R10, R13, R3, R4, R5, R6, R8, R9: 10k, Resistor_SMD:R_0402_1005Metric, symbol Device:R
- added R11, R12, R7: 10R, Resistor_SMD:R_0402_1005Metric, symbol Device:R
- added TP1: G, TestPoint:TestPoint_Pad_D1.5mm, symbol Connector:TestPoint
- added TP2: 3, TestPoint:TestPoint_Pad_D1.5mm, symbol Connector:TestPoint
- added TP3: 5, TestPoint:TestPoint_Pad_D1.5mm, symbol Connector:TestPoint
- added TP4: H, TestPoint:TestPoint_Pad_D1.5mm, symbol Connector:TestPoint
- added TP5: L, TestPoint:TestPoint_Pad_D1.5mm, symbol Connector:TestPoint
- added TP6: T, TestPoint:TestPoint_Pad_D1.5mm, symbol Connector:TestPoint
- added TP7: R, TestPoint:TestPoint_Pad_D1.5mm, symbol Connector:TestPoint
- added TP8: A, TestPoint:TestPoint_Pad_D1.5mm, symbol Connector:TestPoint
- added TP9: B, TestPoint:TestPoint_Pad_D1.5mm, symbol Connector:TestPoint
- added U1: STM32L432KBUx, Package_DFN_QFN:QFN-32-1EP_5x5mm_P0.5mm_EP3.45x3.45mm, symbol MCU_ST_STM32L4:STM32L432KBUx
- added U2: XC6206P332MR-G, Package_TO_SOT_SMD:SOT-23-3, symbol Regulator_Linear:XC6206PxxxMR
- added U3: SIT1050TK, Package_DFN_QFN:DFN-8-1EP_3x3mm_P0.65mm_EP1.5x2.25mm, symbol USER:SIT1050TK
- J1, J2: value AudioJack4_SwitchT1 -> XB-PJ-1837; MPN (none) -> XB-PJ-1837
- J3: MPN (none) -> 2328702-8
Connections:
- net +3.3V: now also C1.2, C4.2, C5.2, C6.2, C68.2, J4.10 (Pin_10), J5.1 (Pin_1), Q2.4 (S), R13.1, R8.1, TP2.1, U1.1 (VDD), U1.17 (VDD), U1.5 (VDDA), U2.2 (VO)
- net +5V: now also C3.2, C73.2, F1.1, R3.1, TP3.1, U2.3 (VI), U3.3 (VCC); no longer J1.4, J2.4
- net GND: now also C1.1, C2.1, C3.1, C4.1, C5.1, C6.1, C68.1, C7.1, C73.1, D1.3 (A), J4.11 (Pin_11), J4.13 (Pin_13), J4.8 (Pin_8), J5.3 (Pin_3), Q2.1 (S), R10.2, R4.2, R6.2, TP1.1, U1.16 (VSS), U1.32 (VSS), U1.33 (VSS), U2.1 (GND), U3.2 (GND), U3.8 (S)
- net LCD_CS: now also J4.7 (Pin_7), U1.10 (PA4)
- net LCD_RES: now also J4.6 (Pin_6), U1.8 (PA2)
- net LCD_RS: now also J4.5 (Pin_5), U1.9 (PA3)
- net LCD_SCL: now also J4.4 (Pin_4), U1.11 (PA5)
- net LCD_SDA: now also J4.3 (Pin_3), U1.13 (PA7)
- net at J3.1 (Pin_1): now also J4.12 (Pin_12), R7.2
- net CAN_L: now reaches J1.2, J2.2
- net CAN_L: now also D1.2 (K), R2.1, TP5.1, U3.6 (CANL)
- net CAN_H: now reaches J1.3, J2.3
- net CAN_H: now also D1.1 (K), R1.2, TP4.1, U3.7 (CANH)
- net at J2.5: now also R5.1
- net at J1.5: now also R9.1
- new net: Q2.6 (D), Q3.2 (G), R3.2
- new net: R11.1, U3.1 (TXD)
- new net: C2.2, Q3.1 (S), Q3.4 (S), U3.5 (VREF)
- new net: F1.2, J1.4, J2.4
- new net: R12.1, U3.4 (RXD)
- new net: Q3.6 (D), R1.1
- new net: Q3.3 (D), R2.2
- new net: Q2.3 (D), R7.1
- new net CAN_RX: R12.2, TP7.1, U1.21 (PA11)
- new net CAN_TERM: Q2.2 (G), Q3.5 (G), R4.1, U1.19 (PA9)
- new net CAN_TX: R11.2, TP6.1, U1.22 (PA12)
- new net DET_A: R5.2, R6.1, TP8.1, U1.6 (PA0)
- new net DET_B: R10.1, R9.2, TP9.1, U1.7 (PA1)
- new net LCD_PWM: Q2.5 (G), R8.2, U1.18 (PA8)
- new net NRST: C7.2, J5.2 (Pin_2), R13.2, U1.4 (NRST)
- new net SWC: J5.4 (Pin_4), U1.24 (PA14)
- new net SWD: J5.5 (Pin_5), U1.23 (PA13)
- no-connect marks 0 -> 3
Other:
- title: (none) -> Headunit
- moved on the sheet: J1, J2, J3
