File: Gearunit/HW_Gearunit/Board/PWR.kicad_sch (KiCad schematic)
At the start: 45 parts, among them J3 Keystone 590, J4 TYPE-C-31-E-08, J6 Keystone 590, Q4 AO3400A, Q5 AO3400A, U10 FUSB302BMPX, U2 XC6206P332MR-G, U7 TPS61023DRLR, U8 BQ24259RGER, U9 DW01A

Commit message: Gearunit updates, Readme updated
Parts:
- added C21, C22: 100n, Capacitor_SMD:C_0402_1005Metric, symbol Device:C
- added R21, R22, R23: 10k, Resistor_SMD:R_0402_1005Metric, symbol Device:R
- added R48: 30k, Resistor_SMD:R_0603_1608Metric, symbol Device:R
- added U12: INA181A1IDBV, Package_TO_SOT_SMD:SOT-23-6, symbol Amplifier_Current:INA181
- R20: renamed from R48; value 30k -> 100mR; MPN 0603WAF3002T5E -> ERJ3RSFR10V
- R70: footprint Resistor_SMD:R_0603_1608Metric -> Resistor_SMD:R_0402_1005Metric; MPN 0603WAF1502T5E -> 0402WGF1502TCE
Connections:
- net +3.3V: now also C21.1, R22.2, R23.1, U12.6 (V+)
- net BAT_INT: now also R23.2
- net GND: now also C21.2, R21.1, R48.1, U12.2 (GND); no longer R20.1
- net VBAT: now also R20.2, C22.1, U12.3 (+); no longer J6.1 (Pin_1), R8.2
- net at R47.2, TH2.1, U8.11 (TS): now also R48.2; no longer R20.2
- new net: R21.2, R22.1, U12.5 (REF)
- new net BAT_I: U12.1
- new net BAT_V: C22.2, J6.1 (Pin_1), R20.1, R8.2, U12.4 (-)
Other:
- moved on the sheet: C1, C64, C65, C66, C73, D2, J3, J6, L13, R17, R20, R70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
